File: hardware/kicad/tinySensorv1.sch (KiCad schematic (older format))
At the start: 19 parts, among them J1 RADIO, J10 CR2032 socket, J11 AAA socket, J12 AA Socket, J13 Bornier, J2 DCDC converter, J3 BMP/BME breakout, J5 OneWire sensor, J6 ISP, J7 Analog sensor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

Commit message: Create new 'library' folder for footprints
Parts:
- J2: footprint Chinese breakouts:DC-DC 0.9v-3.3v to 3.3v -> TinySensor lib:DC-DC_0.9v-3.3v_to_3.3v
- J3: footprint Chinese breakouts:BMx280 breakout -> TinySensor lib:BMx280_breakout
- J6: footprint Connector_PinHeader_2.54mm:PinHeader_2x03_P2.54mm_Vertical -> TinySensor lib:AVR_ICSP
Changed lines of the file:
@@
 F 0 "J3" H 6950 4700 50  0000 L CNN
 F 1 "BMP/BME breakout" H 6950 4600 50  0000 L CNN
-F 2 "Chinese breakouts:BMx280 breakout" H 6800 4650 50  0001 C CNN
+F 2 "TinySensor lib:BMx280_breakout" H 6800 4650 50  0001 C CNN
 F 3 "~" H 6800 4650 50  0001 C CNN
 	1    6800 4650
@@
 F 0 "J6" H 1970 4396 50  0000 R CNN
 F 1 "ISP" H 1970 4305 50  0000 R CNN
-F 2 "Connector_PinHeader_2.54mm:PinHeader_2x03_P2.54mm_Vertical" V 2000 4350 50  0001 C CNN
+F 2 "TinySensor lib:AVR_ICSP" V 2000 4350 50  0001 C CNN
 F 3 " ~" H 975 3750 50  0001 C CNN
 	1    2250 4300
@@
 F 0 "J2" H 6979 1242 50  0000 L CNN
 F 1 "DCDC converter" H 6979 1151 50  0000 L CNN
-F 2 "Chinese breakouts:DC-DC 0.9v-3.3v to 3.3v" H 6900 1200 50  0001 C CNN
+F 2 "TinySensor lib:DC-DC_0.9v-3.3v_to_3.3v" H 6900 1200 50  0001 C CNN
 F 3 "~" H 6900 1200 50  0001 C CNN
 	1    6900 1200

Commit message: Updated card layout
* Use new ICSP footprint
* Better capacitor footprint
* board limits
* removed all tracks, to be refined
Parts:
- removed C3: 0.1n, Capacitor_THT:CP_Radial_Tantal_D4.5mm_P2.50mm, symbol Device:C
- C2: footprint Capacitor_THT:C_Rect_L10.0mm_W4.0mm_P7.50mm_FKS3_FKP3 -> Capacitor_THT:C_Rect_L7.0mm_W2.0mm_P5.00mm
- J6: footprint TinySensor lib:AVR_ICSP -> TinySensor lib:ICSP_SOCKET_MINI_2x3
Connections:
- wire segments 85 -> 81
Changed lines of the file:
@@
 F 0 "C2" V 6248 2150 50  0000 C CNN
 F 1 "100n" V 6339 2150 50  0000 C CNN
-F 2 "Capacitor_THT:C_Rect_L10.0mm_W4.0mm_P7.50mm_FKS3_FKP3" H 6538 2000 50  0001 C CNN
+F 2 "Capacitor_THT:C_Rect_L7.0mm_W2.0mm_P5.00mm" H 6538 2000 50  0001 C CNN
 F 3 "~" H 6500 2150 50  0001 C CNN
 	1    6500 2150
@@
 F 0 "J6" H 1970 4396 50  0000 R CNN
 F 1 "ISP" H 1970 4305 50  0000 R CNN
-F 2 "TinySensor lib:AVR_ICSP" V 2000 4350 50  0001 C CNN
+F 2 "TinySensor lib:ICSP_SOCKET_MINI_2x3" V 2000 4350 50  0001 C CNN
 F 3 " ~" H 975 3750 50  0001 C CNN
 	1    2250 4300
@@
 $EndComp
 Wire Wire Line
-	4700 4550 5400 4550
-$Comp
-L Device:C C3
-U 1 1 5BCD88C5
-P 5250 4300
-F 0 "C3" V 4998 4300 50  0000 C CNN
-F 1 "0.1n" V 5089 4300 50  0000 C CNN
-F 2 "Capacitor_THT:CP_Radial_Tantal_D4.5mm_P2.50mm" H 5288 4150 50  0001 C CNN
-F 3 "~" H 5250 4300 50  0001 C CNN
-	1    5250 4300
-	0    1    1    0
-$EndComp
-Wire Wire Line
 	6000 3750 6000 4450
 Wire Wire Line
 	5750 3850 5750 4550
-Wire Wire Line
-	5400 4300 5400 4550
-Connection ~ 5400 4550
-Wire Wire Line
-	5100 4300 5100 4450
-Wire Wire Line
-	4700 4450 5100 4450
-Connection ~ 5100 4450
-Wire Wire Line
-	5100 4450 6000 4450
 Connection ~ 6000 4450
 Wire Wire Line
 	6000 4450 6600 4450
-Wire Wire Line
-	5400 4550 5750 4550
 Connection ~ 5750 4550
 Wire Wire Line
 	5750 4550 6600 4550
+Wire Wire Line
+	4700 4550 5750 4550
+Wire Wire Line
+	4700 4450 6000 4450
 $EndSCHEMATC

Commit message: Finish a first version of PCB layout
Parts:
- removed J3: BMP/BME breakout, TinySensor lib:BMx280_breakout, symbol Connector_Generic_MountingPin:Conn_01x06_MountingPin
- added C3: 1u, Capacitor_THT:CP_Radial_D4.0mm_P1.50mm, symbol Device:CP1
- added J3: BMP/BME breakout, TinySensor lib:BMx280_breakout, symbol Connector:Conn_01x06_Female
- added JP2: Direct alim, Connector_PinHeader_2.54mm:PinHeader_1x02_P2.54mm_Vertical, symbol Device:Jumper
- added R4: 75R, Resistor_THT:R_Axial_DIN0204_L3.6mm_D1.6mm_P7.62mm_Horizontal, symbol Device:R
- added R6: 4k7, Resistor_THT:R_Axial_DIN0204_L3.6mm_D1.6mm_P7.62mm_Horizontal, symbol Device:R
Connections:
- net labels added: +3V3, PWM_OUT
- wire segments 81 -> 90
- no-connect marks 5 -> 3
Other:
- moved on the sheet: J10, J11, J12, J13

Commit message: Initial hardware version (first batch)
Parts:
- removed JP2: Direct alim, Connector_PinHeader_2.54mm:PinHeader_1x02_P2.54mm_Vertical, symbol Device:Jumper
- added C4: 1n, Capacitor_THT:CP_Radial_Tantal_D4.5mm_P2.50mm, symbol Device:C_Small
- added JP2: DIRECT Vcc, Jumper:SolderJumper-2_P1.3mm_Open_TrianglePad1.0x1.5mm, symbol Jumper:SolderJumper_2_Open
- added MH1, MH2, MH3, MH4, MH5, MH6, MH7: MountingHole, MountingHole:MountingHole_2.5mm, symbol Mechanical:MountingHole
Connections:
- wire segments 90 -> 93
Other:
- note added: "Optional RC filter for LM35 sensor"
- note added: "Radio activity led"
- moved on the sheet: C3, D1, JP1, R1, R4
