File: hardware/kicad/tinySensorv1.sch (KiCad schematic (older format))
At the start: 30 parts, among them J1 RADIO, J10 CR2032 socket, J11 AAA socket, J12 AA Socket, J13 Bornier, J2 DCDC converter, J3 BMP/BME breakout, J5 OneWire sensor, J6 ISP, J7 Analog sensor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

Commit message: Merge overlapping traces, add a 1n capacitor after DCDC converter
Parts:
- added C2: 100n, Capacitor_THT:C_Rect_L7.0mm_W2.0mm_P5.00mm, symbol Device:C
- C5: renamed from C2; value 100n -> 1n; footprint Capacitor_THT:C_Rect_L7.0mm_W2.0mm_P5.00mm -> Capacitor_THT:CP_Radial_Tantal_D4.5mm_P2.50mm
Connections:
- wire segments 93 -> 95
Other:
- moved on the sheet: C1
Changed lines of the file:
@@
 L Device:CP C1
 U 1 1 5BCDDA39
-P 6500 1700
-F 0 "C1" V 6755 1700 50  0000 C CNN
-F 1 "10u" V 6664 1700 50  0000 C CNN
-F 2 "Capacitor_THT:CP_Radial_D5.0mm_P2.50mm" H 6538 1550 50  0001 C CNN
-F 3 "~" H 6500 1700 50  0001 C CNN
-	1    6500 1700
-	0    -1   -1   0
-$EndComp
-Wire Wire Line
-	6650 1700 6650 1200
+P 6500 1550
+F 0 "C1" V 6550 1450 50  0000 C CNN
+F 1 "10u" V 6500 1250 50  0000 C CNN
+F 2 "Capacitor_THT:CP_Radial_D5.0mm_P2.50mm" H 6538 1400 50  0001 C CNN
+F 3 "~" H 6500 1550 50  0001 C CNN
+	1    6500 1550
+	0    -1   -1   0
+$EndComp
 Connection ~ 6650 1200
 Wire Wire Line
 	6650 1200 6700 1200
-Wire Wire Line
-	6350 1700 6350 1300
 Connection ~ 6350 1300
 Wire Wire Line
 	6350 1300 6700 1300
 $Comp
-L Device:C C2
+L Device:C C5
 U 1 1 5BCDF3E0
 P 6500 2150
-F 0 "C2" V 6248 2150 50  0000 C CNN
-F 1 "100n" V 6339 2150 50  0000 C CNN
-F 2 "Capacitor_THT:C_Rect_L7.0mm_W2.0mm_P5.00mm" H 6538 2000 50  0001 C CNN
+F 0 "C5" V 6450 2250 50  0000 C CNN
+F 1 "1n" V 6500 2400 50  0000 C CNN
+F 2 "Capacitor_THT:CP_Radial_Tantal_D4.5mm_P2.50mm" H 6538 2000 50  0001 C CNN
 F 3 "~" H 6500 2150 50  0001 C CNN
 	1    6500 2150
 	0    1    1    0
 $EndComp
-Connection ~ 6650 1700
-Connection ~ 6350 1700
-Wire Wire Line
-	6650 1700 6650 2150
-Wire Wire Line
-	6350 1700 6350 2150
 Text Notes 10200 2300 0    50   ~ 0
 Power management
@@
 Wire Wire Line
 	4900 4650 5200 4650
+$Comp
+L Device:C C2
+U 1 1 5BEB17B5
+P 6500 1850
+F 0 "C2" V 6450 1950 50  0000 C CNN
+F 1 "100n" V 6500 2150 50  0000 C CNN
+F 2 "Capacitor_THT:C_Rect_L7.0mm_W2.0mm_P5.00mm" H 6538 1700 50  0001 C CNN
+F 3 "~" H 6500 1850 50  0001 C CNN
+	1    6500 1850
+	0    1    1    0
+$EndComp
+Connection ~ 6350 1550
+Connection ~ 6650 1550
+Wire Wire Line
+	6650 1200 6650 1550
+Wire Wire Line
+	6350 1300 6350 1550
+Connection ~ 6650 1850
+Wire Wire Line
+	6650 1850 6650 2150
+Connection ~ 6350 1850
+Wire Wire Line
+	6350 1850 6350 2150
+Wire Wire Line
+	6350 1550 6350 1850
+Wire Wire Line
+	6650 1550 6650 1850
 $EndSCHEMATC

Commit message: Alpha of pcb version 2
Parts:
- added J4: PWM_OUT, Connector_PinHeader_2.54mm:PinHeader_1x01_P2.54mm_Vertical, symbol Connector:Conn_01x01_Female
- J13: value Bornier -> RAW IN
Connections:
- net labels added: SENSOR_VCC, VCC
- net labels removed: +3.3V, +3V3
- wire segments 95 -> 91
- no-connect marks 3 -> 2
Other:
- note added: "Bypass of DC-DC converter"
- note removed: "(LM35)"
- moved on the sheet: J10, J11, J12, J13, JP2

Commit message: Fix HW bugs around analog sensor and begin radio connector move
Parts:
- U1: symbol MCU_Microchip_ATtiny:ATtiny84A-PU -> tinySensorv1-rescue:ATtiny84A-PU-MCU_Microchip_ATtiny
Connections:
- wire segments 91 -> 92
Changed lines of the file:
@@
 $EndComp
 $Comp
-L MCU_Microchip_ATtiny:ATtiny84A-PU U1
+L tinySensorv1-rescue:ATtiny84A-PU-MCU_Microchip_ATtiny U1
 U 1 1 5BCB880C
 P 2250 2000
@@
 	-1   0    0    1
 $EndComp
-Text Label 5200 4650 0    50   ~ 0
+Text Label 5050 4550 0    50   ~ 0
 Analog_sensor
 $Comp
@@
 Wire Wire Line
 	6000 4450 6600 4450
-Connection ~ 5750 4550
 Wire Wire Line
 	5750 4550 6600 4550
-Wire Wire Line
-	4700 4550 5750 4550
 Wire Wire Line
 	4700 4450 6000 4450
@@
 	0    -1   -1   0
 $EndComp
-Wire Wire Line
-	4700 4650 4900 4650
-Wire Wire Line
-	4900 4950 4900 4650
-Connection ~ 4900 4650
-Wire Wire Line
-	4900 4650 5200 4650
 $Comp
 L Device:C C2
@@
 Wire Wire Line
 	9850 1650 10400 1650
+Wire Wire Line
+	5750 4650 5750 4550
+Connection ~ 5750 4550
+Wire Wire Line
+	4700 4550 4900 4550
+Wire Wire Line
+	4700 4650 5750 4650
+Wire Wire Line
+	4900 4950 4900 4550
+Connection ~ 4900 4550
+Wire Wire Line
+	4900 4550 5050 4550
 $EndSCHEMATC

Commit message: Use new DCDC converter footprint, do no explicitely display GND
Parts:
- U1: symbol tinySensorv1-rescue:ATtiny84A-PU-MCU_Microchip_ATtiny -> tinySensorv1-rescue:ATtiny84A-PU-MCU_Microchip_ATtiny-tinySensorv1-rescue
Changed lines of the file:
@@
 $EndComp
 $Comp
-L tinySensorv1-rescue:ATtiny84A-PU-MCU_Microchip_ATtiny U1
+L tinySensorv1-rescue:ATtiny84A-PU-MCU_Microchip_ATtiny-tinySensorv1-rescue U1
 U 1 1 5BCB880C
 P 2250 2000
@@
 	2850 2100 3350 2100
 Wire Wire Line
-	9050 1550 9050 1750
-Connection ~ 9050 1750
-Wire Wire Line
 	10300 1550 10300 1750
 Wire Wire Line
 	10400 1550 10400 1650
-Wire Wire Line
-	9150 1550 9150 1650
-Connection ~ 9150 1650
 $Comp
 L power:GND #PWR0117
@@
 	10300 1750 10300 1850
 Wire Wire Line
-	9050 1750 9750 1750
-Wire Wire Line
-	9150 1650 9450 1650
-Wire Wire Line
 	8000 1650 8250 1650
 Wire Wire Line
@@
 	9750 1750 10300 1750
 Wire Wire Line
-	8450 1550 8450 1750
-Wire Wire Line
-	8450 1750 9050 1750
-Wire Wire Line
 	8000 1650 8000 1350
 Connection ~ 8250 1650
-Wire Wire Line
-	8250 1650 8550 1650
 Wire Wire Line
 	8250 1950 7850 1950
@@
 Connection ~ 4900 1100
 Wire Wire Line
-	8550 1550 8550 1650
-Connection ~ 8550 1650
-Wire Wire Line
-	8550 1650 9150 1650
-Wire Wire Line
 	9850 1550 9850 1650
 Connection ~ 9850 1650
@@
 Wire Wire Line
 	4900 4550 5050 4550
+Wire Wire Line
+	8250 1650 8450 1650
+Wire Wire Line
+	8550 1550 8550 1750
+Wire Wire Line
+	8450 1550 8450 1650
+Connection ~ 8450 1650
+Wire Wire Line
+	8450 1650 9050 1650
+Wire Wire Line
+	8550 1750 9150 1750
+Wire Wire Line
+	9050 1550 9050 1650
+Connection ~ 9050 1650
+Wire Wire Line
+	9050 1650 9450 1650
+Wire Wire Line
+	9150 1550 9150 1750
+Connection ~ 9150 1750
+Wire Wire Line
+	9150 1750 9750 1750
 $EndSCHEMATC

Commit message: Update new board and Readme
Parts:
- removed C4: 1n, Capacitor_THT:CP_Radial_Tantal_D4.5mm_P2.50mm, symbol Device:C_Small
- removed J4: PWM_OUT, Connector_PinHeader_2.54mm:PinHeader_1x01_P2.54mm_Vertical, symbol Connector:Conn_01x01_Female
- added C4: 10u, Capacitor_THT:CP_Radial_D5.0mm_P2.50mm, symbol Device:CP
- added J4: PWM out, Connector_PinHeader_2.54mm:PinHeader_1x02_P2.54mm_Vertical, symbol Connector:Conn_01x02_Male
Connections:
- wire segments 92 -> 93
Changed lines of the file:
@@
 	4050 3250 4050 6200
-$Comp
-L Device:C_Small C4
-U 1 1 5BE98657
-P 8800 3850
-F 0 "C4" V 8571 3850 50  0000 C CNN
-F 1 "1n" V 8662 3850 50  0000 C CNN
-F 2 "Capacitor_THT:CP_Radial_Tantal_D4.5mm_P2.50mm" H 8800 3850 50  0001 C CNN
-F 3 "~" H 8800 3850 50  0001 C CNN
-	1    8800 3850
-	0    1    1    0
-$EndComp
 $Comp
 L power:GND #PWR0123
 U 1 1 5BE989C1
-P 9050 3850
-F 0 "#PWR0123" H 9050 3600 50  0001 C CNN
-F 1 "GND" H 9055 3677 50  0000 C CNN
-F 2 "" H 9050 3850 50  0001 C CNN
-F 3 "" H 9050 3850 50  0001 C CNN
-	1    9050 3850
+P 9150 3850
+F 0 "#PWR0123" H 9150 3600 50  0001 C CNN
+F 1 "GND" H 9155 3677 50  0000 C CNN
+F 2 "" H 9150 3850 50  0001 C CNN
+F 3 "" H 9150 3850 50  0001 C CNN
+	1    9150 3850
 	1    0    0    -1
 $EndComp
 Wire Wire Line
 	8600 3850 8700 3850
-Wire Wire Line
-	8900 3850 9050 3850
 $Comp
 L Mechanical:MountingHole MH6
@@
 	-1   0    0    1
 $EndComp
-$Comp
-L Connector:Conn_01x01_Female J4
-U 1 1 5BEAA179
-P 3550 2100
-F 0 "J4" H 3578 2126 50  0000 L CNN
-F 1 "PWM_OUT" H 3700 2100 50  0000 L CNN
-F 2 "Connector_PinHeader_2.54mm:PinHeader_1x01_P2.54mm_Vertical" H 3550 2100 50  0001 C CNN
-F 3 "~" H 3550 2100 50  0001 C CNN
-	1    3550 2100
-	1    0    0    -1
-$EndComp
 Wire Wire Line
 	5950 1300 6350 1300
-Wire Wire Line
-	2850 2100 3350 2100
 Wire Wire Line
 	10300 1550 10300 1750
@@
 Wire Wire Line
 	9150 1750 9750 1750
+$Comp
+L Device:CP C4
+U 1 1 5E0B7120
+P 8850 3850
+F 0 "C4" V 8950 3700 50  0000 C CNN
+F 1 "10u" V 9014 3850 50  0000 C CNN
+F 2 "Capacitor_THT:CP_Radial_D5.0mm_P2.50mm" H 8888 3700 50  0001 C CNN
+F 3 "~" H 8850 3850 50  0001 C CNN
+	1    8850 3850
+	0    -1   -1   0
+$EndComp
+Wire Wire Line
+	9150 3850 9000 3850
+$Comp
+L Connector:Conn_01x02_Male J4
+U 1 1 5E0CE887
+P 4050 2200
+F 0 "J4" H 4156 2378 50  0000 C CNN
+F 1 "PWM out" H 4156 2287 50  0000 C CNN
+F 2 "Connector_PinHeader_2.54mm:PinHeader_1x02_P2.54mm_Vertical" H 4050 2200 50  0001 C CNN
+F 3 "~" H 4050 2200 50  0001 C CNN
+	1    4050 2200
+	-1   0    0    1
+$EndComp
+Wire Wire Line
+	2850 2100 3850 2100
+$Comp
+L power:GND #PWR0101
+U 1 1 5E0E2B34
+P 3700 2200
+F 0 "#PWR0101" H 3700 1950 50  0001 C CNN
+F 1 "GND" H 3705 2027 50  0000 C CNN
+F 2 "" H 3700 2200 50  0001 C CNN
+F 3 "" H 3700 2200 50  0001 C CNN
+	1    3700 2200
+	1    0    0    -1
+$EndComp
+Wire Wire Line
+	3700 2200 3850 2200
 $EndSCHEMATC

Commit message: feat: Many updates of PCB
* Fixed many polarity bugs: Vcc is always on the square pad, but
  for 433Mhz emmiter which is somewhat strange
* Added INT0 header
* Allow resistor bridge on analog sensor, to allow usage of LDR
Parts:
- removed MH7: MountingHole, MountingHole:MountingHole_2.5mm, symbol Mechanical:MountingHole
- added J8: EXT. INT0, Connector_PinHeader_2.54mm:PinHeader_1x02_P2.54mm_Vertical, symbol Connector_Generic:Conn_01x02
- added JP3: (no value), Jumper:SolderJumper-2_P1.3mm_Open_TrianglePad1.0x1.5mm, symbol Jumper:SolderJumper_2_Open
- J3: value BMP/BME breakout -> I2C Sensor (BME/BMP 280)
- J6: symbol Connector:AVR-ISP-6 -> tinySensorv1-rescue:AVR-ISP-6-Connector
Connections:
- net labels added: INT0
- wire segments 93 -> 102
- no-connect marks 2 -> 1
Other:
- note added: "Optional RC filter for LM35 sensor \nor resistor bridge for LDR"
- note removed: "Optional RC filter for LM35 sensor"
- moved on the sheet: D1, J4, R6
Changed lines of the file:
@@
 EESchema Schematic File Version 4
-LIBS:tinySensorv1-cache
-EELAYER 26 0
+EELAYER 30 0
 EELAYER END
 $Descr A4 11693 8268
@@
 Sheet 1 1
 Title "TinySensor board"
-Date "2018-11-12"
+Date "2020-06-28"
 Rev "2.0"
 Comp ""
@@
 F 3 "~" H 2800 6350 50  0001 C CNN
 	1    2800 6350
-	-1   0    0    1
+	1    0    0    -1
 $EndComp
 $Comp
@@
 Wire Wire Line
 	6600 1100 6700 1100
-NoConn ~ 2850 2500
 $Comp
 L power:GND #PWR0105
@@
 F 3 "~" H 6500 2150 50  0001 C CNN
 	1    6500 2150
-	0    1    1    0
+	0    -1   -1   0
 $EndComp
 Text Notes 10200 2300 0    50   ~ 0
@@
 	2850 2600 3000 2600
 $Comp
-L Connector:AVR-ISP-6 J6
+L tinySensorv1-rescue:AVR-ISP-6-Connector J6
 U 1 1 5BCF975A
 P 2250 4300
@@
 U 1 1 5BD28967
 P 4500 4550
-F 0 "J7" H 4900 4450 50  0000 C CNN
-F 1 "Analog sensor" H 4900 4550 50  0000 C CNN
+F 0 "J7" H 4650 4550 50  0000 C CNN
+F 1 "Analog sensor" H 4500 4800 50  0000 C CNN
 F 2 "Connector_PinHeader_2.54mm:PinHeader_1x03_P2.54mm_Vertical" H 4500 4550 50  0001 C CNN
 F 3 "~" H 4500 4550 50  0001 C CNN
@@
 U 1 1 5BD3495A
 P 5050 3850
-F 0 "J5" H 5450 3800 50  0000 C CNN
-F 1 "OneWire sensor" H 5450 3900 50  0000 C CNN
+F 0 "J5" H 5200 3850 50  0000 C CNN
+F 1 "OneWire sensor" H 5050 4100 50  0000 C CNN
 F 2 "Connector_PinHeader_2.54mm:PinHeader_1x03_P2.54mm_Vertical" H 5050 3850 50  0001 C CNN
 F 3 "~" H 5050 3850 50  0001 C CNN
@@
 	5750 3500 5750 3850
 Wire Wire Line
-	5250 3750 6000 3750
-Connection ~ 6000 3750
-Wire Wire Line
 	5250 3850 5750 3850
 Connection ~ 5750 3850
-Text Label 5400 3950 0    50   ~ 0
-OneWire
 Wire Notes Line
 	4050 3250 7750 3250
@@
 $EndComp
 Wire Wire Line
-	6000 3750 6000 4200
-Wire Wire Line
-	5750 3850 5750 4550
-Connection ~ 6000 4450
+	5750 3850 5750 4450
 Wire Wire Line
 	6000 4450 6600 4450
 Wire Wire Line
 	5750 4550 6600 4550
-Wire Wire Line
-	4700 4450 6000 4450
 Wire Wire Line
 	2850 2300 3000 2300
@@
 P 6800 4650
 F 0 "J3" H 6827 4626 50  0000 L CNN
-F 1 "BMP/BME breakout" H 6827 4535 50  0000 L CNN
+F 1 "I2C Sensor (BME/BMP 280)" H 6250 4200 50  0000 L CNN
 F 2 "TinySensor lib:BMx280_breakout" H 6800 4650 50  0001 C CNN
 F 3 "~" H 6800 4650 50  0001 C CNN
@@
 L power:GND #PWR0120
 U 1 1 5BDB0112
-P 4900 5550
-F 0 "#PWR0120" H 4900 5300 50  0001 C CNN
-F 1 "GND" H 5000 5400 50  0000 R CNN
-F 2 "" H 4900 5550 50  0001 C CNN
-F 3 "" H 4900 5550 50  0001 C CNN
-	1    4900 5550
+P 4900 5600
+F 0 "#PWR0120" H 4900 5350 50  0001 C CNN
+F 1 "GND" H 5000 5450 50  0000 R CNN
+F 2 "" H 4900 5600 50  0001 C CNN
+F 3 "" H 4900 5600 50  0001 C CNN
+	1    4900 5600
 	1    0    0    -1
 $EndComp
@@
 L Device:R R6
 U 1 1 5BDB363C
-P 5400 4200
-F 0 "R6" V 5193 4200 50  0000 C CNN
-F 1 "4k7" V 5284 4200 50  0000 C CNN
-F 2 "Resistor_THT:R_Axial_DIN0204_L3.6mm_D1.6mm_P7.62mm_Horizontal" V 5330 4200 50  0001 C CNN
-F 3 "~" H 5400 4200 50  0001 C CNN
-	1    5400 4200
+P 5400 3600
+F 0 "R6" V 5193 3600 50  0000 C CNN
+F 1 "4k7" V 5284 3600 50  0000 C CNN
+F 2 "Resistor_THT:R_Axial_DIN0204_L3.6mm_D1.6mm_P7.62mm_Horizontal" V 5330 3600 50  0001 C CNN
+F 3 "~" H 5400 3600 50  0001 C CNN
+	1    5400 3600
 	0    1    1    0
 $EndComp
-Wire Wire Line
-	5550 4200 6000 4200
-Connection ~ 6000 4200
-Wire Wire Line
-	6000 4200 6000 4450
-Wire Wire Line
-	5250 4200 5250 3950
-Connection ~ 5250 3950
-Wire Wire Line
-	5250 3950 5400 3950
 Wire Notes Line
 	5850 2400 11000 2400
@@
 Wire Notes Line rgb(0, 194, 0)
 	4450 4950 5800 4950
-Text Notes 4450 5850 0    50   ~ 0
-Optional RC filter for LM35 sensor
-Wire Notes Line rgb(0, 194, 0)
-	4450 5950 5800 5950
+Text Notes 4500 5950 0    50   ~ 0
+Optional RC filter for LM35 sensor \nor resistor bridge for LDR
 Wire Notes Line rgb(114, 194, 0)
-	5800 4950 5800 5950
+	5950 4950 5950 5950
 Wire Notes Line rgb(0, 194, 0)
 	4450 4950 4450 5950
@@
 F 3 "~" H 10150 5150 50  0001 C CNN
 	1    10150 5150
-	0    -1   -1   0
-$EndComp
-$Comp
-L Mechanical:MountingHole MH7
-U 1 1 5BEA80BA
-P 10350 5150
-F 0 "MH7" H 10450 5196 50  0000 L CNN
-F 1 "MountingHole" H 10450 5105 50  0000 L CNN
-F 2 "MountingHole:MountingHole_2.5mm" H 10350 5150 50  0001 C CNN
-F 3 "~" H 10350 5150 50  0001 C CNN
-	1    10350 5150
 	0    -1   -1   0
 $EndComp
@@
 Text Label 6000 3400 0    50   ~ 0
 SENSOR_VCC
-Wire Wire Line
-	6000 3400 6000 3750
 $Comp
 L power:VCC #PWR05
@@
 Wire Wire Line
 	5950 1300 6350 1300
-Wire Wire Line
-	10300 1550 10300 1750
-Wire Wire Line
-	10400 1550 10400 1650
 $Comp
 L power:GND #PWR0117
@@
 	1    0    0    -1
 $EndComp
-Connection ~ 10300 1750
 Wire Wire Line
 	10300 1750 10300 1850
 Wire Wire Line
 	8000 1650 8250 1650
-Wire Wire Line
-	9750 1550 9750 1750
-Connection ~ 9750 1750
-Wire Wire Line
-	9750 1750 10300 1750
 Wire Wire Line
 	8000 1650 8000 1350
@@
 	9450 850  9450 1650
 Connection ~ 9450 1650
-Wire Wire Line
-	9450 1650 9850 1650
 Text Notes 7700 2100 0    50   ~ 0
 Bypass of DC-DC converter
@@
 Connection ~ 4900 1100
 Wire Wire Line
-	9850 1550 9850 1650
-Connection ~ 9850 1650
-Wire Wire Line
-	9850 1650 10400 1650
-Wire Wire Line
-	5750 4650 5750 4550
-Connection ~ 5750 4550
-Wire Wire Line
 	4700 4550 4900 4550
-Wire Wire Line
-	4700 4650 5750 4650
 Wire Wire Line
 	4900 4950 4900 4550
@@
 	9150 1550 9150 1750
 Connection ~ 9150 1750
-Wire Wire Line
-	9150 1750 9750 1750
 $Comp
 L Device:CP C4
@@
 	9150 3850 9000 3850
 $Comp
+L power:GND #PWR0101
+U 1 1 5E0E2B34
+P 4150 2100
+F 0 "#PWR0101" H 4150 1850 50  0001 C CNN
+F 1 "GND" H 4155 1927 50  0000 C CNN
+F 2 "" H 4150 2100 50  0001 C CNN
+F 3 "" H 4150 2100 50  0001 C CNN
+	1    4150 2100
+	1    0    0    -1
+$EndComp
+$Comp
+L Jumper:SolderJumper_2_Open JP3
+U 1 1 5EF9D131
+P 5450 5450
+F 0 "JP3" V 5450 5200 50  0000 L CNN
+F 1 " " V 5350 4950 50  0000 L CNN
+F 2 "Jumper:SolderJumper-2_P1.3mm_Open_TrianglePad1.0x1.5mm" H 5450 5450 50  0001 C CNN
+F 3 "~" H 5450 5450 50  0001 C CNN
+	1    5450 5450
+	0    -1   -1   0
+$EndComp
+Wire Wire Line
+	5450 5600 4900 5600
+Wire Wire Line
+	4900 5550 4900 5600
+Connection ~ 4900 5600
+Wire Notes Line rgb(7, 194, 0)
+	5800 4950 5950 4950
+Wire Wire Line
+	4900 5250 5450 5250
+Wire Wire Line
+	5450 5250 5450 5300
+Wire Notes Line rgb(0, 194, 0)
+	4450 5950 5950 5950
+Connection ~ 4900 5250
+$Comp
+L Connector_Generic:Conn_01x02 J8
+U 1 1 5F04FEAF
+P 2200 5450
+F 0 "J8" H 2280 5442 50  0000 L CNN
+F 1 "EXT. INT0" H 1800 5650 50  0000 L CNN
+F 2 "Connector_PinHeader_2.54mm:PinHeader_1x02_P2.54mm_Vertical" H 2200 5450 50  0001 C CNN
+F 3 "~" H 2200 5450 50  0001 C CNN
+	1    2200 5450
+	1    0    0    -1
+$EndComp
+$Comp
+L power:GND #PWR0103
+U 1 1 5F052C10
+P 2000 5600
+F 0 "#PWR0103" H 2000 5350 50  0001 C CNN
+F 1 "GND" H 2005 5427 50  0000 C CNN
+F 2 "" H 2000 5600 50  0001 C CNN
+F 3 "" H 2000 5600 50  0001 C CNN
+	1    2000 5600
+	1    0    0    -1
+$EndComp
+Wire Wire Line
+	2000 5550 2000 5600
+Text Label 1700 5450 0    50   ~ 0
+INT0
+Wire Wire Line
+	1700 5450 2000 5450
+Wire Wire Line
+	2850 2500 3000 2500
+Text Label 3000 2500 0    50   ~ 0
+INT0
+Wire Wire Line
+	4700 4450 5750 4450
+Connection ~ 5750 4450
+Wire Wire Line
+	5750 4450 5750 4550
+Wire Wire Line
+	6000 4450 6000 4650
+Wire Wire Line
+	6000 4650 4700 4650
+Connection ~ 6000 4450
+Wire Wire Line
+	9450 1650 9750 1650
+Wire Wire Line
+	10300 1550 10300 1650
+Wire Wire Line
+	9750 1550 9750 1650
+Connection ~ 9750 1650
+Wire Wire Line
+	9750 1650 10300 1650
+Wire Wire Line
+	9150 1750 9850 1750
+Connection ~ 10300 1750
+Wire Wire Line
+	10300 1750 10400 1750
+Wire Wire Line
+	10400 1550 10400 1750
+Wire Wire Line
+	9850 1550 9850 1750
+Connection ~ 9850 1750
+Wire Wire Line
+	9850 1750 10300 1750
+Wire Wire Line
+	2850 2100 3900 2100
+Wire Wire Line
+	6000 3400 6000 3600
+Wire Wire Line
+	5550 3600 6000 3600
+Connection ~ 6000 3600
+Wire Wire Line
+	5250 3600 5250 3750
+Wire Wire Line
+	6000 3600 6000 3950
+Wire Wire Line
+	5250 3750 5350 3750
+Connection ~ 5250 3750
+Text Label 5350 3750 0    50   ~ 0
+OneWire
+Wire Wire Line
+	5250 3950 6000 3950
+Connection ~ 6000 3950
+Wire Wire Line
+	6000 3950 6000 4450
+$Comp
 L Connector:Conn_01x02_Male J4
 U 1 1 5E0CE887
-P 4050 2200
-F 0 "J4" H 4156 2378 50  0000 C CNN
-F 1 "PWM out" H 4156 2287 50  0000 C CNN
-F 2 "Connector_PinHeader_2.54mm:PinHeader_1x02_P2.54mm_Vertical" H 4050 2200 50  0001 C CNN
-F 3 "~" H 4050 2200 50  0001 C CNN
-	1    4050 2200
-	-1   0    0    1
-$EndComp
-Wire Wire Line
-	2850 2100 3850 2100
-$Comp
-L power:GND #PWR0101
-U 1 1 5E0E2B34
-P 3700 2200
-F 0 "#PWR0101" H 3700 1950 50  0001 C CNN
-F 1 "GND" H 3705 2027 50  0000 C CNN
-F 2 "" H 3700 2200 50  0001 C CNN
-F 3 "" H 3700 2200 50  0001 C CNN
-	1    3700 2200
-	1    0    0    -1
-$EndComp
-Wire Wire Line
-	3700 2200 3850 2200
+P 3900 2300
+F 0 "J4" H 4006 2478 50  0000 C CNN
+F 1 "PWM out" V 3800 2250 50  0000 C CNN
+F 2 "Connector_PinHeader_2.54mm:PinHeader_1x02_P2.54mm_Vertical" H 3900 2300 50  0001 C CNN
+F 3 "~" H 3900 2300 50  0001 C CNN
+	1    3900 2300
+	0    -1   -1   0
+$EndComp
+Wire Wire Line
+	4150 2100 4000 2100
+Connection ~ 4150 2100
+Connection ~ 4000 2100
 $EndSCHEMATC
