File: hardware/tinysensor/tinySensorv1.kicad_sch (KiCad schematic)
At the start: 39 parts, among them J1 RADIO, J10 CR2032 socket, J11 AAA socket, J12 AA Socket, J13 RAW IN, J2 DCDC converter, J3 I2C Sensor (BME/BMP 280), J4 Digital out, J5 OneWire sensor, J6 ISP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

Commit message: hardware: Update of Kikad design, new batch expected
Parts:
- removed R5: 10k, Resistor_THT:R_Axial_DIN0204_L3.6mm_D1.6mm_P7.62mm_Horizontal, symbol Device:R
